File: amplifier.sch (EAGLE design)
At the start: 7 parts

Commit message: Saving
Connections:
- net N$1 renamed BRIDGE_A
- net N$3 renamed BRIDGE_C
- new net BRIDGE_D: B1.+
Changed lines of the file:
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@@
 </segment>
 </net>
-<net name="N$1" class="0">
+<net name="BRIDGE_A" class="0">
 <segment>
 <pinref part="B1" gate="G$1" pin="AC1"/>
 <wire x1="55.88" y1="114.3" x2="55.88" y2="111.76" width="0.1524" layer="91"/>
-<wire x1="40.64" y1="114.3" x2="55.88" y2="114.3" width="0.1524" layer="91"/>
+<wire x1="40.64" y1="114.3" x2="53.34" y2="114.3" width="0.1524" layer="91"/>
 <pinref part="C1" gate="G$1" pin="2"/>
+<wire x1="53.34" y1="114.3" x2="55.88" y2="114.3" width="0.1524" layer="91"/>
 <wire x1="40.64" y1="111.76" x2="40.64" y2="114.3" width="0.1524" layer="91"/>
 <pinref part="S1" gate="G$1" pin="B"/>
@@
 <wire x1="55.88" y1="114.3" x2="68.58" y2="114.3" width="0.1524" layer="91"/>
 <junction x="55.88" y="114.3"/>
+<label x="53.34" y="119.38" size="1.778" layer="95" rot="R90" xref="yes"/>
+<wire x1="53.34" y1="119.38" x2="53.34" y2="114.3" width="0.1524" layer="91"/>
+<junction x="53.34" y="114.3"/>
 </segment>
 </net>
@@
 </segment>
 </net>
-<net name="N$3" class="0">
+<net name="BRIDGE_C" class="0">
 <segment>
 <pinref part="D15" gate="G$1" pin="C"/>
@@
 <wire x1="50.8" y1="106.68" x2="48.26" y2="106.68" width="0.1524" layer="91"/>
 <wire x1="48.26" y1="106.68" x2="48.26" y2="93.98" width="0.1524" layer="91"/>
-<wire x1="48.26" y1="93.98" x2="96.52" y2="93.98" width="0.1524" layer="91"/>
+<wire x1="48.26" y1="93.98" x2="53.34" y2="93.98" width="0.1524" layer="91"/>
+<wire x1="53.34" y1="93.98" x2="96.52" y2="93.98" width="0.1524" layer="91"/>
 <wire x1="96.52" y1="93.98" x2="96.52" y2="114.3" width="0.1524" layer="91"/>
+<label x="53.34" y="88.9" size="1.778" layer="95" rot="R270" xref="yes"/>
+<wire x1="53.34" y1="88.9" x2="53.34" y2="93.98" width="0.1524" layer="91"/>
+<junction x="53.34" y="93.98"/>
 </segment>
 </net>
+<net name="BRIDGE_D" class="0">
+<segment>
+<pinref part="B1" gate="G$1" pin="+"/>
+<wire x1="60.96" y1="106.68" x2="78.74" y2="106.68" width="0.1524" layer="91"/>
+<label x="83.82" y="106.68" size="1.778" layer="95" xref="yes"/>
+<wire x1="78.74" y1="106.68" x2="78.74" y2="83.82" width="0.1524" layer="91"/>
+<wire x1="78.74" y1="106.68" x2="83.82" y2="106.68" width="0.1524" layer="91"/>
+<junction x="78.74" y="106.68"/>
+</segment>
+</net>

Commit message: Finished 70%
Parts:
- added C11: 470pF, rcl:C-EUC0603
- added C12, C13: .22uF, rcl:C-EUC0603
- added C2, C34: 0.01uF, rcl:C-EUC0603
- added C20: .022uF, rcl:C-EUC0603
- added C21: .033uF, rcl:C-EUC0603
- added C22: 100pF, rcl:C-EUC0603
- added C23, C24: 22uF, resistor:CPOL-USE10-30
- added C25, C32, C33: 1kuF, resistor:CPOL-USE10-30
- added C26: 0.1uF, rcl:C-EUC0603
- added C30: 220uF, resistor:CPOL-USE3.5-8
- added C31: 0.22uF, rcl:C-EUC0603
- added C8: .001uF, rcl:C-EUC0603
- added D1, D6, D7, D8: (no value), adafruit:DIODESOD-323F
- added D10, D3, D9: 1N4004, diode:1N4004
- added J8: 47R, rcl:R-US_R0603
- added Q7, Q8, T1: 2N2222, adafruit:2N2222
- added R1, R48: 220R, rcl:R-US_R0603
- added R16, R18: 2k7, rcl:R-US_R0603
- added R17: 47k, rcl:R-US_R0603
- added R19: 8k2, rcl:R-US_R0603
- added R2, VR3, VR4, VR5, VR6: PC16S, piher:PC16S
- added R20: 10k, rcl:R-US_R0603
- added R21, R22, R35: 100k, rcl:R-US_R0603
- added R30, R34: 470k, rcl:R-US_R0603
- added R31: 150k, rcl:R-US_R0603
- added R32: 1k5, rcl:R-US_R0603
- added R36, R38: 68k, rcl:R-US_R0603
- added R37: 82k, rcl:R-US_R0603
- added R39: 330R, rcl:R-US_R0603
- added R40: 2k4, rcl:R-US_R0603
- added R41: 0R1, rcl:R-US_R0603
- added R42: 4R7, rcl:R-US_R0603
- added R43: 100R, rcl:R-US_R0603
- C1: value (none) -> 1kuF; device rcl:C-EUC0603 -> resistor:CPOL-USE10-30
- R49: value (none) -> 3k3
Connections:
- new net GND: C23.-, C31.1, C8.1, D10.A, D8.A, J8.2, R18.2, R30.2, R39.1, R43.2, VR3.1E, VR4.1A, VR4.1S, VR5.1A, VR5.1S
- new net N$1: C30.+, R31.2, R48.2
- new net N$10: C11.2, R17.1, VR6.1A
- new net N$11: C11.1, R19.1
- new net N$12: C12.1, R16.2, R17.2
- new net N$13: C12.2, C13.2, R19.2
- new net N$14: C13.1, R18.1, VR5.1E
- new net N$15: R20.1, VR6.1S
- new net N$16: C21.2, R20.2, R21.1, R22.1
- new net N$17: C21.1, C22.1, D7.A, D8.C, R36.2, VR6.1E
- new net N$18: R22.2
- new net N$19: R21.2
- new net N$20: R16.1, VR4.1E
- new net N$21: C24.+, R38.1
- new net N$22: R38.2
- new net N$23: C8.2, R34.1, VR3.1A
- new net N$24: C20.2, R34.2
- new net N$25: R32.1, VR3.1S
- new net N$26: Q8.E, R32.2
- new net N$28: Q7.E, Q8.B, R30.1
- new net N$29: D6.A, Q7.B
- new net N$3: C22.2, C23.+, D7.C, R35.2, R36.1, R37.2
- new net N$30: D6.C
- new net N$31: C20.1, Q7.C, Q8.C, R31.1
- new net N$4: R40.1, R41.1
- new net N$5: C24.-, R39.2, R40.2
- new net N$6: C26.2, R42.1
- new net N$7: C25.-, R42.2
- new net N$8: C25.+, D10.C, D9.A
- new net N$9: R43.1
- net BRIDGE_A: now also C34.2; no longer C1.2
- net BRIDGE_C: now also C26.1, C30.-, C32.-, C33.-, J8.1, R37.1, R41.2
- net BRIDGE_D: now also C31.2, C32.+, C33.+, D9.C, R35.1, R48.1
- net V-: now also C34.1; no longer C1.1
Other:
- note added: "GND from C"
- note added: "Middle Jack - Sleeve + Housing"
- note added: "NOT finished"
- note added: "Notes: 1. High Power Rs: R41; R43; J8 2. D9;D10 are currently through hole - could be changed 3. J5; C31 - are not directly connected, could be connected with a metalic plae (heat sink) 4. SP+ is currently NOT on the schematics 5. C8 - the value is unknown"
- note added: "Possibly AGND"
- note added: "To HPhone Jack - Ring + Housing"
- note added: "To IC1 Pin 4 (OUTPUT)"
- note added: "To IC1 Pin1"
- note added: "To IC1 Pin2"
- note added: "To IC1 Pin3"
- note added: "To IC1 Pin4"
- note added: "To IC1 Pin5"
- note added: "To Middle Jack - Ring Shunt Spring"
- note added: "To Middle Jack - Tip Shunt Spring"
- note added: "To SP-"
- note added: "To Shunt side of HPhone Jack"
